Commit message: update the origin value of object

File: hrwros_assignment2.xacro (robot description, xacro)
@@ -80,5 +80,5 @@
   </link>
   <joint name="sphere_joint" type="fixed">
-    <origin xyz="5.9 -4.6 0" />
+    <origin xyz="5.9 -4.6 0.4" />
     <parent link="world" />
     <child link="sphere_link" />
